File: pcb/matrix.kicad_sch (KiCad schematic)
At the start: 158 parts

Commit message: update to latest
Parts:
- added MX1: CL, PCM_marbastlib-mx:SW_MX_1.25u, symbol marbastlib-mx:MX_SW_solder
Connections:
- net COL03: now also MX1.1
- net at D1.2 (A), MX1.2: now also MX1.2
Changed lines of the file:
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@@
   (junction (at 53.34 33.02) (diameter 0) (color 0 0 0 0)
   )
+  (junction (at 58.42 55.88) (diameter 0) (color 0 0 0 0)
+  )
   (junction (at 123.19 43.18) (diameter 0) (color 0 0 0 0)
   )
@@
     (stroke (width 0) (type default))
   )
+  (wire (pts (xy 53.34 50.8) (xy 56.515 50.8))
+    (stroke (width 0) (type default))
+  )
   (wire (pts (xy 146.05 43.18) (xy 157.48 43.18))
     (stroke (width 0) (type default))
@@
   )
   (wire (pts (xy 232.41 33.02) (xy 232.41 50.8))
+    (stroke (width 0) (type default))
+  )
+  (wire (pts (xy 58.42 55.88) (xy 61.595 55.88))
     (stroke (width 0) (type default))
   )
@@
     )
   )
+  (symbol (lib_id "marbastlib-mx:MX_SW_solder") (at 59.055 53.34 0) (unit 1)
+    (in_bom no) (on_board yes) (dnp no) (fields_autoplaced)
+    (property "Reference" "MX1" (at 59.055 45.72 0)
+      (effects (font (size 1.27 1.27)))
+    )
+    (property "Value" "CL" (at 59.055 48.26 0)
+      (effects (font (size 1.27 1.27)))
+    )
+    (property "Footprint" "PCM_marbastlib-mx:SW_MX_1.25u" (at 59.055 53.34 0)
+      (effects (font (size 1.27 1.27)) hide)
+    )
+    (property "Datasheet" "~" (at 59.055 53.34 0)
+      (effects (font (size 1.27 1.27)) hide)
+    )
+    (pin "1")
+    (pin "2")
+    (instances
+      (project "matrix"
+        (path "/2b21a88c-dcce-4c32-b74d-cb04a08504d3"
+          (reference "MX1") (unit 1)
+        )
+      )
+      (project "spell"
+        (path "/45a14dd6-89f9-47c6-b9b2-743a88e53966/5d1fa359-692b-42ab-9b17-0d321cb6a293"
+          (reference "MX81") (unit 1)
+        )
+      )
+      (project "ice60v2"
+        (path "/98d602aa-46a9-4e45-be3d-3b1e6175f1d0/737834b9-aee7-4cf4-b31e-7e166d45723a"
+          (reference "MX10") (unit 1)
+        )
+      )
+    )
+  )
   (symbol (lib_id "marbastlib-mx:MX_SW_solder") (at 55.88 109.22 0) (unit 1)
     (in_bom no) (on_board yes) (dnp no) (fields_autoplaced)
@@
   )
   (symbol (lib_id "marbastlib-mx:MX_SW_solder") (at 55.88 53.34 0) (unit 1)
-    (in_bom no) (on_board yes) (dnp no) (fields_autoplaced)
+    (in_bom no) (on_board yes) (dnp no)
     (property "Reference" "MX1" (at 55.88 45.72 0)
       (effects (font (size 1.27 1.27)))
