File: pcb/spell.kicad_pcb (KiCad board)
At the start: 2 copper layers, 360.8 x 75.1 mm, 182 parts, among them J1 JST SH 4p, SW1 RST, SW2 BOOT, U1 STM32F072CBTx, U2 XC6206PxxxMR

Commit message: update to latest
Parts:
- added MX81: CL, PCM_marbastlib-mx:SW_MX_1.25u, F.Cu at (87.5, 56.6)
- moved C3 0.86 mm to (332.9, 71.4)
- moved C6 0.86 mm to (332.9, 70.2)
Routing:
- net +3V3: track 53.4 -> 47.8 mm
- net Net-(D21-A): track 3.69 -> 8.46 mm
- net COL03: track 316.0 -> 320.7 mm
- net GND: track 41.5 -> 37.4 mm, vias 21 -> 24
- net ~{RST}: track 22.7 -> 23.5 mm
